Commit message: urdf plus extra view

File: newton/examples/assets/a1_description/urdf/robot.urdf (robot description, URDF)
Before this commit: robot a1, 33 links, 32 joints
Links:
- link camera_bottom_screw_frame: mass None -> 0.001
- link camera_link: mass 0.564 -> 0.200

File: newton/examples/assets/a1_description/xacro/_d435.urdf.xacro (robot description, xacro)
@@ -29,5 +29,11 @@
             <child link="${name}_bottom_screw_frame" />
         </joint>
-        <link name="${name}_bottom_screw_frame" />
+        <link name="${name}_bottom_screw_frame" ">
+            <inertial>
+                <mass value="0.001"/>
+                <origin rpy="0 0 0" xyz="0 0 0"/>
+                <inertia ixx="0.0001" ixy="0" ixz="0" iyy="0.0001" iyz="0" izz="0.0001"/>
+            </inertial>
+        </link>
         <joint name="${name}_link_joint" type="fixed">
             <origin xyz="0 ${d435_cam_depth_py} ${d435_cam_depth_pz}" rpy="0 0 0" />
@@ -55,8 +61,7 @@
             <inertial>
                 <!-- The following are not reliable values, and should not be used for modeling -->
-                <mass value="0.564" />
+                <mass value="0.200" />
                 <origin xyz="0 0 0" />
-                <inertia ixx="0.003881243" ixy="0.0" ixz="0.0" iyy="0.000498940" iyz="0.0"
-                    izz="0.003879257" />
+                <inertia ixx="2.083e-5" ixy="0.0" ixz="0.0" iyy="1.452e-4" iyz="0.0" izz="1.452e-4" />
             </inertial>
         </link>
